File: Hardware/Basic/Top/NotSoSmartWatch-BASIC-TOP.sch (EAGLE design)
At the start: 51 parts, among them U2 NRF52832_MODULE_MDBT42, U4 PCF8523

Commit message: updated through Take 002
Parts:
- added C22: 100n, LinnesLab-Passives:CAPACITOR0603
- added C23, C24: 47p, LinnesLab-Passives:CAPACITOR0603
- added J1: (no value), LinnesLab-Connectors:CONN_07
- added JP2: (no value), LinnesLab-Switches:JUMPER-SMT_2_NO_SILK
- added LED5: RED, LinnesLab-LED:LED0603
- added LED6: YELLOW, LinnesLab-LED:LED0603
- added R1, R2: 0, LinnesLab-Passives:RESISTOR0603
- added R17, R18: 27, LinnesLab-Passives:RESISTOR0603
- added R19, R20: 1k, LinnesLab-Passives:RESISTOR0603
- added U5: FT231XS, LinnesLab-DigitalIC:FT231XS
- renumbered U$1 to SW1, U$2 to SW2
Connections:
- removed net BATT: R13.1, R14.2
- removed net CD1: SD2.CARD_DETECT
- removed net CHRG.STAT: CHRG2.STAT, R12.1
- removed net CS.OLED: U3./CS
- removed net DC.OLED: U3.DC/I2C_SA0
- removed net RESET.OLED: U3./RES
- removed net RXD: U2.P0.08
- removed net SD.CS: SD2.CS
- removed net SW1: SW1.1, SW2.1
- removed net TXD: U2.P0.06
- removed net VBATT: U4.VBAT
- new net !CTS: JP2.2, U5.!CTS
- new net !DTR: U5.!DTR
- new net A4/VBATT: R13.1, R14.2, U2.P0.28/AIN4
- new net A6/TIA: J1.7, U2.P0.30/AIN6
- new net A7/PPG: J1.5, U2.P0.31/AIN7
- new net D11/SW1: SW1.1, U2.P0.11
- new net D15/SW2: SW2.1, U2.P0.15
- new net D16/CS.OLED: U2.P0.16, U3./CS
- new net D27/CHRG.STAT: CHRG2.STAT, R12.1, U2.P0.27
- new net D29/LED.CTRL: J1.6, U2.P0.29/AIN5
- new net D3/RESET.OLED: U2.P0.03/AIN1, U3./RES
- new net D4/DC.OLED: U2.P0.04/AIN2, U3.DC/I2C_SA0
- new net D5/CD1: SD2.CARD_DETECT, U2.P0.05/AIN3
- new net D7/SD.CS: SD2.CS, U2.P0.07
- new net FT3V3: U5.3V3OUT
- new net N$23: R17.2, U5.USBDM
- new net N$24: R18.2, U5.USBDP
- new net N$25: LED5.C, R19.2
- new net N$26: LED6.C, R20.2
- new net RXD.FT: R2.1, U5.RXD
- new net RXD.NRF: R1.2, U2.P0.08
- new net RXLED: R19.1, U5.CBUS1
- new net TXD.FT: R1.1, U5.TXD
- new net TXD.NRF: R2.2, U2.P0.06
- new net TXLED: R20.1, U5.CBUS2
- net 3.3V: now also C22.2, J1.2, LED5.A, LED6.A, U5.!RESET, U5.VCCIO
- net GND: now also C22.1, C23.2, C24.1, J1.1, JP2.1, U5.GND@16, U5.GND@6
- net SCL: now also J1.3, R9.1; no longer R8.1
- net SDA: now also J1.4, R8.1; no longer R9.1
- net USB+: now also C23.1, R18.1
- net USB-: now also C24.2, R17.1
- net V_USB: now also U5.VCC
Other:
- note added: "FTDI Serial-to-USB"
- note added: "Header Pins"
- note added: "I don't remember if CTS needs to be grounded or left floating so here's a jumper to ground so it can be configued either way dynamically."
- note added: "TXD goes to RX on the other device RXD goes to TX on the other device"
- moved on the sheet: C10, C11, C8, C9, R8, R9, SW4, XTAL2

Commit message: updated through Take 003
Parts:
- removed C22: 100n, LinnesLab-Passives:CAPACITOR0603
- removed C23, C24: 47p, LinnesLab-Passives:CAPACITOR0603
- removed D4: (no value), LinnesLab-DiscreteSemi:SCHOTTKY-USC
- removed LED5: RED, LinnesLab-LED:LED0603
- removed LED6: YELLOW, LinnesLab-LED:LED0603
- removed R19: 1k, LinnesLab-Passives:RESISTOR0603
- removed U3: (no value), LinnesLab-Displays:DISP_OLED_UG-2864HSWEG01-NO-WRAPAROUND
- removed XTAL3: 32.7680kHz, LinnesLab-Clocks:CRYSTALECS-.327-12.5-12-C-TR
- added C1: 1u, LinnesLab-Passives:CAPACITOR0603
- added C3, C4: (no value), LinnesLab-Passives:CAPACITOR0603
- added D3: (no value), LinnesLab-DiscreteSemi:SCHOTTKY-USC
- added LED1: RED, LinnesLab-LED:LED0603
- added LED2: BLUE, LinnesLab-LED:LED0603
- added R10: 10k, LinnesLab-Passives:RESISTOR0603
- added RTC: PCF8523, LinnesLab-Clocks:PCF8523
- added XTAL1: 32.768kHz, LinnesLab-Clocks:CRYSTALECS-.327-12.5-12-C-TR
- C10: value 300p -> 4.7u
- C11: value 300p -> 100n
- C12: value 10u -> 47p; device LinnesLab-Passives:CAPACITOR0805 -> LinnesLab-Passives:CAPACITOR0603; SPICEPREFIX (none) -> C
- C13: value 2.2uF -> 47p; device LinnesLab-Passives:CAPACITOR0402 -> LinnesLab-Passives:CAPACITOR0603; SPICEPREFIX (none) -> C
- C14: SPICEPREFIX (none) -> C
- C15: value 2.2uF -> 10uF; device LinnesLab-Passives:CAPACITOR0402 -> LinnesLab-Passives:CAPACITOR0603
- C16: value 10uF -> 2.2uF; device LinnesLab-Passives:CAPACITOR0603 -> LinnesLab-Passives:CAPACITOR0402
- C2: value 1u -> 10u; device LinnesLab-Passives:CAPACITOR0603 -> LinnesLab-Passives:CAPACITOR0805
- C20: value 4.7u -> 2.2uF; device LinnesLab-Passives:CAPACITOR0603 -> LinnesLab-Passives:CAPACITOR0402
- C21: value 4.7u -> 1u
- C5, C6: value 1u -> 300p
- C7: value 1u -> 4.7u
- C8, C9: value (none) -> 1u
- J1: device LinnesLab-Connectors:CONN_07 -> LinnesLab-Connectors:CONN_07-1.27MM
- LED3: SPICEPREFIX (none) -> L
- LED4: value BLUE -> YELLOW; SPICEPREFIX (none) -> L
- R1, R2: value 0 -> 10k
- R11: value (none) -> 27; SPICEPREFIX (none) -> R
- R12: value 100k -> 27; SPICEPREFIX (none) -> R
- R13: value 100k -> 10k
- R14: value 100k -> 1k; SPICEPREFIX (none) -> R
- R15: value 100k -> 390k
- R17, R18: value 27 -> 0; SPICEPREFIX R -> (none)
- R3: value 1k -> 100k
- R5: value 10k -> 1k
- R6: value 10k -> (none)
- R7: value 390k -> 100k
- R8, R9: value 10k -> 100k
- SW1, SW2: value SWITCH.MOM -> (none); device LinnesLab-Switches:SWITCH.MOM -> LinnesLab-Switches:SPST-PTS830GG140-COPY.1-3
- SW3, SW4: value (none) -> SWITCH.MOM; device LinnesLab-Switches:SPST-PTS830GG140-COPY.1-3 -> LinnesLab-Switches:SWITCH.MOM
- U4: value PCF8523 -> (none); device LinnesLab-Clocks:PCF8523 -> LinnesLab-Displays:DISP_OLED_UG-2864HSWEG01-NO-WRAPAROUND; DIGIKEY 568-5306-1-ND -> (none); I2C_ADDRESS 0x68h -> (none); MFN PCF8523T/1,118 -> (none); MFN_MANUFACTURER NXP USA Inc. -> (none)
- XTAL2: value 32.768kHz -> 32.7680kHz; FREQ (none) -> 32.7680KHZ
- renumbered CHRG2 to CHRG, CORTEX1 to DEBUG1, D5 to D2, JP2 to JP1, L2 to L1, LDO2 to LDO1, R20 to R16, SD2 to SD1, U2 to U1, U5 to FTDI, USB2 to USB1
Connections:
- new net N$21: J1.5
- new net N$22: J1.4
- new net N$27: J1.3
- new net N$28: J1.2
- new net N$29: J1.1
- net 3.3V: now also C14.2, C2.2, C20.2, C21.1, C9.1, D3.C, J1.7, LED3.A, LED4.A, R1.2, R10.2, R2.2, R7.2, RTC.VDD, U4.VBAT; no longer C12.2, C17.2, C2.1, C22.2, C6.1, D1.C, J1.2, LED5.A, LED6.A, R15.2, R5.2, R8.2, R9.2, U3.VBAT, U3.VDD
- net A4/VBATT: now also R8.1, R9.2; no longer R13.1, R14.2
- net A6/TIA: no longer J1.7
- net A7/PPG: no longer J1.5
- net D11/SW1: now also SW3.1; no longer SW1.1
- net D15/SW2: now also SW4.1; no longer SW2.1
- net D16/CS.OLED: now also U4./CS; no longer U3./CS
- net D27/CHRG.STAT: now also R3.1; no longer R12.1
- net D29/LED.CTRL: no longer J1.6
- net D3/RESET.OLED: now also U4./RES; no longer U3./RES
- net D4/DC.OLED: now also U4.DC/I2C_SA0; no longer U3.DC/I2C_SA0
- net DFU: now also SW1.B; no longer SW3.B
- net DTR: now also C11.1; no longer C14.1
- net GND: now also C1.2, C13.2, C14.1, C15.1, C2.1, C20.1, C21.2, C3.1, C4.2, C5.2, C7.1, J1.6, LED1.C, LED2.C, R13.1, R15.2, R7.1, R9.1, RTC.VSS, SW1.A, SW2.B, SW3.3, SW3.4, SW4.3, SW4.4, U4.BS0, U4.BS2, U4.NC(GND)@1, U4.NC(GND)@2, U4.VLSS; no longer C11.2, C16.1, C18.1, C2.2, C20.2, C21.1, C22.1, C23.2, C24.1, C5.1, C7.2, J1.1, LED3.C, LED4.C, R11.1, R14.1, R15.1, R7.2, SW1.3, SW1.4, SW2.3, SW2.4, SW3.A, SW4.B, U3.BS0, U3.BS2, U3.NC(GND)@1, U3.NC(GND)@2, U3.VLSS, U3.VSS
- net LED1: now also R4.2; no longer R3.2
- net LED2: now also R5.2; no longer R4.2
- net MOSI: now also U4.D1/SPI_SDIN/I2C_SDA; no longer U3.D1/SPI_SDIN/I2C_SDA
- net N$1: now also R13.2, U4.BS1; no longer R6.2, U3.BS1
- net N$10: now also LED2.A, R5.1; no longer LED4.A, R4.1
- net N$12: now also C1.1; no longer C7.1
- net N$13: now also C15.2, U4.VCC; no longer C16.2, U3.VCC
- net N$15: now also C17.2, U4.VCOMH; no longer C18.2, U3.VCOMH
- net N$17: now also R6.2; no longer R11.2
- net N$19: now also RTC.OSCO, XTAL2.1; no longer U4.OSCO, XTAL3.1
- net N$2: now also R15.1, U4.IREF; no longer R7.1, U3.IREF
- net N$20: now also RTC.OSCI, XTAL2.2; no longer U4.OSCI, XTAL3.2
- net N$23: now also R11.2; no longer R17.2
- net N$24: now also R12.2; no longer R18.2
- net N$25: now also LED3.C, R14.2; no longer LED5.C, R19.2
- net N$26: now also LED4.C; no longer LED6.C
- net N$3: now also C18.2, U4.C2P; no longer C13.2, U3.C2P
- net N$4: now also C3.2, XTAL1.1; no longer C8.2, XTAL2.1
- net N$5: now also C18.1, U4.C2N; no longer C13.1, U3.C2N
- net N$6: now also C4.1, XTAL1.2; no longer C9.1, XTAL2.2
- net N$7: now also C16.2, U4.C1P; no longer C15.2, U3.C1P
- net N$8: now also C16.1, U4.C1N; no longer C15.1, U3.C1N
- net N$9: now also LED1.A, R4.1; no longer LED3.A, R3.1
- net P0.09/NFC1: now also C5.1; no longer C11.1
- net P0.10/NFC2: now also C6.1; no longer C10.1
- net RESET: now also C11.2, D3.A, R10.1, SW2.A; no longer C14.2, D1.A, R5.1, SW4.A
- net RXD.FT: now also R18.1; no longer R2.1
- net RXD.NRF: now also R17.2; no longer R1.2
- net RXLED: now also R14.1; no longer R19.1
- net SCK: now also U4.D0/SPI_SCLK/I2C_SCK; no longer U3.D0/SPI_SCLK/I2C_SCK
- net SCL: now also R2.1, RTC.SCL; no longer J1.3, R9.1, U4.SCL
- net SDA: now also R1.1, RTC.SDA; no longer J1.4, R8.1, U4.SDA
- net TXD.FT: now also R17.1; no longer R1.1
- net TXD.NRF: now also R18.2; no longer R2.2
- net USB+: now also C13.1, R12.1; no longer C23.1, R18.1
- net USB-: now also C12.2, R11.1; no longer C24.2, R17.1
- net VIN: now also C7.2, C8.2, D1.C, R3.2; no longer C21.2, C5.2, D4.C, R12.2
- net VLIPO: now also C10.1, D1.A, R8.2; no longer C20.1, D4.A, R13.2
Other:
- moved on the sheet: C10, C11, C12, C13, C14, C15, C16, C17, C18, C2, C20, C21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

Commit message: updated through Take 005
Parts:
- removed C5, C6: 300p, LinnesLab-Passives:CAPACITOR0603
Connections:
- net GND: no longer C5.2, C6.2
- net P0.09/NFC1: no longer C5.1
- net P0.10/NFC2: no longer C6.1
Changed lines of the file:
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@@
 <part name="GND15" library="LinnesLab-Symbols" deviceset="GND" device=""/>
 <part name="GND16" library="LinnesLab-Symbols" deviceset="GND" device=""/>
-<part name="GND17" library="LinnesLab-Symbols" deviceset="GND" device=""/>
-<part name="GND18" library="LinnesLab-Symbols" deviceset="GND" device=""/>
 <part name="GND19" library="LinnesLab-Symbols" deviceset="GND" device=""/>
 <part name="GND20" library="LinnesLab-Symbols" deviceset="GND" device=""/>
@@
 <part name="C3" library="LinnesLab-Passives" deviceset="CAPACITOR" device="0603" package3d_urn="urn:adsk.eagle:package:15661989/2"/>
 <part name="C4" library="LinnesLab-Passives" deviceset="CAPACITOR" device="0603" package3d_urn="urn:adsk.eagle:package:15661989/2"/>
-<part name="C6" library="LinnesLab-Passives" deviceset="CAPACITOR" device="0603" package3d_urn="urn:adsk.eagle:package:15661989/2" value="300p"/>
-<part name="C5" library="LinnesLab-Passives" deviceset="CAPACITOR" device="0603" package3d_urn="urn:adsk.eagle:package:15661989/2" value="300p"/>
 <part name="C2" library="LinnesLab-Passives" deviceset="CAPACITOR" device="0805" package3d_urn="urn:adsk.eagle:package:15662010/2" value="10u"/>
 <part name="L1" library="LinnesLab-Passives" deviceset="INDUCTOR" device="0603" override_package3d_urn="urn:adsk.eagle:package:18592195/2" override_package_urn="urn:adsk.eagle:footprint:18592196/1" value="10u"/>
@@
 <attribute name="VALUE" x="101.6" y="78.486" size="1.778" layer="96" align="top-center"/>
 </instance>
-<instance part="GND17" gate="G$1" x="104.14" y="45.72" smashed="yes">
-<attribute name="VALUE" x="104.14" y="45.466" size="1.778" layer="96" align="top-center"/>
-</instance>
-<instance part="GND18" gate="G$1" x="91.44" y="45.72" smashed="yes">
-<attribute name="VALUE" x="91.44" y="45.466" size="1.778" layer="96" align="top-center"/>
-</instance>
 <instance part="GND19" gate="G$1" x="81.28" y="45.72" smashed="yes">
 <attribute name="VALUE" x="81.28" y="45.466" size="1.778" layer="96" align="top-center"/>
@@
 <attribute name="NAME" x="82.804" y="56.261" size="1.778" layer="95"/>
 <attribute name="VALUE" x="82.804" y="51.181" size="1.778" layer="96"/>
-</instance>
-<instance part="C6" gate="G$1" x="104.14" y="53.34" smashed="yes">
-<attribute name="NAME" x="105.664" y="56.261" size="1.778" layer="95"/>
-<attribute name="VALUE" x="105.664" y="51.181" size="1.778" layer="96"/>
-</instance>
-<instance part="C5" gate="G$1" x="91.44" y="53.34" smashed="yes">
-<attribute name="NAME" x="92.964" y="56.261" size="1.778" layer="95"/>
-<attribute name="VALUE" x="92.964" y="51.181" size="1.778" layer="96"/>
 </instance>
 <instance part="C2" gate="G$1" x="60.96" y="91.44" smashed="yes" rot="R180">
@@
 <pinref part="GND20" gate="G$1" pin="GND"/>
 <pinref part="C3" gate="G$1" pin="1"/>
-</segment>
-<segment>
-<pinref part="C5" gate="G$1" pin="2"/>
-<pinref part="GND18" gate="G$1" pin="GND"/>
-<wire x1="91.44" y1="48.26" x2="91.44" y2="50.8" width="0.1524" layer="91"/>
-</segment>
-<segment>
-<pinref part="C6" gate="G$1" pin="2"/>
-<pinref part="GND17" gate="G$1" pin="GND"/>
-<wire x1="104.14" y1="48.26" x2="104.14" y2="50.8" width="0.1524" layer="91"/>
 </segment>
 <segment>
@@
 <segment>
 <wire x1="96.52" y1="83.82" x2="96.52" y2="60.96" width="0.1524" layer="91"/>
-<wire x1="91.44" y1="60.96" x2="96.52" y2="60.96" width="0.1524" layer="91"/>
-<wire x1="91.44" y1="60.96" x2="91.44" y2="58.42" width="0.1524" layer="91"/>
-<pinref part="C5" gate="G$1" pin="1"/>
 <pinref part="U1" gate="G$1" pin="P0.09"/>
 <label x="96.52" y="63.5" size="1.27" layer="95" rot="R180" xref="yes"/>
@@
 <segment>
 <wire x1="99.06" y1="83.82" x2="99.06" y2="60.96" width="0.1524" layer="91"/>
-<wire x1="99.06" y1="60.96" x2="104.14" y2="60.96" width="0.1524" layer="91"/>
-<wire x1="104.14" y1="60.96" x2="104.14" y2="58.42" width="0.1524" layer="91"/>
-<pinref part="C6" gate="G$1" pin="1"/>
 <pinref part="U1" gate="G$1" pin="P0.10"/>
 <label x="99.06" y="63.5" size="1.27" layer="95" xref="yes"/>
