File: Hardware/Basic/Top/NotSoSmartWatch-BASIC-TOP.brd (EAGLE design)
At the start: 38 x 38 mm, 51 parts, among them U2 NRF52832_MODULE_MDBT42, U4 PCF8523

Commit message: updated through Take 002
Parts:
- added C22: 100n, LinnesLab-Passives:C0603
- added C23, C24: 47p, LinnesLab-Passives:C0603
- added J1: (no value), LinnesLab-Connectors:1X07
- added JP2: (no value), LinnesLab-Switches:SMT-JUMPER_2_NO_SILK
- added LED5: RED, LinnesLab-LED:LED-0603
- added LED6: YELLOW, LinnesLab-LED:LED-0603
- added R1, R2: 0, LinnesLab-Passives:R0603
- added R17, R18: 27, LinnesLab-Passives:R0603
- added R19, R20: 1k, LinnesLab-Passives:R0603
- added U5: FT231XS, LinnesLab-DigitalIC:SSOP20_L
- moved R9 45.3 mm to (-6.43, -12.3), turned to 0 degrees
- moved R8 43.0 mm to (-6.43, -9.60), turned to 0 degrees
- renumbered U$1 to SW1, U$2 to SW2
Connections:
- net VBATT renamed VBAT
- removed net BATT: R13.1, R14.2
- removed net CD1: SD2.CD1
- removed net CHRG.STAT: CHRG2.1, R12.1
- removed net CS.OLED: U3.13
- removed net DC.OLED: U3.15
- removed net RESET.OLED: U3.14
- removed net RXD: U2.21
- removed net SD.CS: SD2.2
- removed net SW1: SW1.A1, SW2.A1
- removed net TXD: U2.19
- new net !CTS: JP2.2, U5.9
- new net !DTR: U5.1
- new net A4/VBATT: R13.1, R14.2, U2.5
- new net A6/TIA: J1.7, U2.7
- new net A7/PPG: J1.5, U2.8
- new net D11/SW1: SW1.A1, U2.25
- new net D15/SW2: SW2.A1, U2.29
- new net D16/CS.OLED: U2.30, U3.13
- new net D27/CHRG.STAT: CHRG2.1, R12.1, U2.4
- new net D29/LED.CTRL: J1.6, U2.6
- new net D3/RESET.OLED: U2.16, U3.14
- new net D4/DC.OLED: U2.17, U3.15
- new net D5/CD1: SD2.CD1, U2.18
- new net D7/SD.CS: SD2.2, U2.20
- new net FT3V3: U5.13
- new net N$23: R17.2, U5.12
- new net N$24: R18.2, U5.11
- new net N$25: LED5.C, R19.2
- new net N$26: LED6.C, R20.2
- new net RXD.FT: R2.1, U5.4
- new net RXD.NRF: R1.2, U2.21
- new net RXLED: R19.1, U5.17
- new net TXD.FT: R1.1, U5.20
- new net TXD.NRF: R2.2, U2.19
- new net TXLED: R20.1, U5.10
- net 3.3V: now also C22.2, J1.2, LED5.A, LED6.A, U5.14, U5.3
- net GND: now also C22.1, C23.2, C24.1, J1.1, JP2.1, U5.16, U5.6
- net SCL: now also J1.3, R9.1; no longer R8.1
- net SDA: now also J1.4, R8.1; no longer R9.1
- net USB+: now also C23.1, R18.1
- net USB-: now also C24.2, R17.1
- net V_USB: now also U5.15

Commit message: updated through Take 003
Parts:
- removed C22: 100n, LinnesLab-Passives:C0603
- removed C23, C24: 47p, LinnesLab-Passives:C0603
- removed CHRG2: MCP73831, LinnesLab-Power:SOT23-5
- removed D4: (no value), LinnesLab-DiscreteSemi:USC
- removed LDO2: MIC5504, LinnesLab-Power:SOT23-5
- removed LED5: RED, LinnesLab-LED:LED-0603
- removed LED6: YELLOW, LinnesLab-LED:LED-0603
- removed R19: 1k, LinnesLab-Passives:R0603
- removed U3: (no value), LinnesLab-Displays:UG-2864HSWEG01_0.96IN_NO-WRAPAROUND
- removed XTAL3: 32.7680kHz, LinnesLab-Clocks:2-SMD.NOLEAD.2.0MMTO1.2MM
- added C1: 1u, LinnesLab-Passives:C0603
- added C3, C4: (no value), LinnesLab-Passives:C0603
- added CHRG: MCP73831, LinnesLab-Power:SOT23-5
- added D3: (no value), LinnesLab-DiscreteSemi:USC
- added LDO1: MIC5504, LinnesLab-Power:SOT23-5
- added LED1: RED, LinnesLab-LED:LED-0603
- added LED2: BLUE, LinnesLab-LED:LED-0603
- added R10: 10k, LinnesLab-Passives:R0603
- added RTC: PCF8523, LinnesLab-Clocks:SO8
- added XTAL1: 32.768kHz, LinnesLab-Clocks:2-SMD.NOLEAD.2.0MMTO1.2MM
- C10: value 300p -> 4.7u
- C11: value 300p -> 100n
- C12: value 10u -> 47p; device LinnesLab-Passives:C0805 -> LinnesLab-Passives:C0603
- C13: value 2.2uF -> 47p; device LinnesLab-Passives:C0402 -> LinnesLab-Passives:C0603
- C15: value 2.2uF -> 10uF; device LinnesLab-Passives:C0402 -> LinnesLab-Passives:C0603
- C16: value 10uF -> 2.2uF; device LinnesLab-Passives:C0603 -> LinnesLab-Passives:C0402
- C2: value 1u -> 10u; device LinnesLab-Passives:C0603 -> LinnesLab-Passives:C0805
- C20: value 4.7u -> 2.2uF; device LinnesLab-Passives:C0603 -> LinnesLab-Passives:C0402
- C21: value 4.7u -> 1u
- C5, C6: value 1u -> 300p
- C7: value 1u -> 4.7u
- C8, C9: value (none) -> 1u
- J1: device LinnesLab-Connectors:1X07 -> LinnesLab-Connectors:1X07_1.27MM
- LED4: value BLUE -> YELLOW
- R1, R2: value 0 -> 10k
- R11: value (none) -> 27
- R12: value 100k -> 27
- R13: value 100k -> 10k
- R14: value 100k -> 1k
- R15: value 100k -> 390k
- R17, R18: value 27 -> 0
- R3: value 1k -> 100k
- R5: value 10k -> 1k
- R6: value 10k -> (none)
- R7: value 390k -> 100k
- R8, R9: value 10k -> 100k
- SW1, SW2: value SWITCH.MOM -> (none); device LinnesLab-Switches:TACTILE_SWITCH_SMD_6.2MM_TALL -> LinnesLab-Switches:BUTTON-GULLWING
- SW3, SW4: value (none) -> SWITCH.MOM; device LinnesLab-Switches:BUTTON-GULLWING -> LinnesLab-Switches:TACTILE_SWITCH_SMD_6.2MM_TALL
- U4: value PCF8523 -> (none); device LinnesLab-Clocks:SO8 -> LinnesLab-Displays:UG-2864HSWEG01_0.96IN_NO-WRAPAROUND
- XTAL2: value 32.768kHz -> 32.7680kHz
- moved R17 72.6 mm to (-6.43, -2.82)
- moved R18 72.4 mm to (-6.43, -5.51)
- moved C11 57.3 mm to (-20.0, 32.6), turned to 270 degrees
- moved R14 57.0 mm to (42.5, 56.9), turned to 0 degrees
- moved R12 53.3 mm to (25.8, 59.3), turned to 0 degrees
- moved R11 52.2 mm to (25.1, 62.6), turned to 0 degrees
- moved XTAL2 50.5 mm to (-1.19, 58.4), turned to 90 degrees
- moved R3 47.6 mm to (20.4, -18.0), turned to 90 degrees
- moved C14 47.2 mm to (38.6, 64.7), turned to 0 degrees
- moved SW2 47.1 mm to (-18.1, 27.9), turned to 180 degrees
- moved C13 46.4 mm to (38.6, 59.7), turned to 0 degrees
- moved R7 46.3 mm to (49.6, -9.88)
- moved D1 41.4 mm to (8.53, 7.04)
- moved C7 41.1 mm to (12.4, -13.3)
- moved LED3 39.3 mm to (42.5, 64.5)
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- renumbered CORTEX1 to DEBUG1, D5 to D2, JP2 to JP1, L2 to L1, R20 to R16, SD2 to SD1, U2 to U1, U5 to FTDI, USB2 to USB1
Connections:
- new net N$21: J1.5
- new net N$22: J1.4
- new net N$27: J1.3
- new net N$28: J1.2
- new net N$29: J1.1
- net 3.3V: now also C14.2, C2.2, C20.2, C21.1, C9.1, D3.-, J1.7, LDO1.5, LED3.A, LED4.A, R1.2, R10.2, R2.2, R7.2, RTC.8, U4.6, U4.9; no longer C12.2, C17.2, C2.1, C22.2, C6.1, D1.-, J1.2, LDO2.5, LED5.A, LED6.A, R15.2, R5.2, R8.2, R9.2, U3.6, U3.9, U4.8
- net A4/VBATT: now also R8.1, R9.2; no longer R13.1, R14.2
- net A6/TIA: no longer J1.7
- net A7/PPG: no longer J1.5
- net D11/SW1: now also SW3.A1; no longer SW1.A1
- net D15/SW2: now also SW4.A1; no longer SW2.A1
- net D16/CS.OLED: now also U4.13; no longer U3.13
- net D27/CHRG.STAT: now also CHRG.1, R3.1; no longer CHRG2.1, R12.1
- net D29/LED.CTRL: no longer J1.6
- net D3/RESET.OLED: now also U4.14; no longer U3.14
- net D4/DC.OLED: now also U4.15; no longer U3.15
- net DFU: now also SW1.3; no longer SW3.3
- net DTR: now also C11.1; no longer C14.1
- net GND: now also C1.2, C13.2, C14.1, C15.1, C2.1, C20.1, C21.2, C3.1, C4.2, C5.2, C7.1, CHRG.2, J1.6, LDO1.2, LED1.C, LED2.C, R13.1, R15.2, R7.1, R9.1, RTC.4, SW1.1, SW2.3, SW3.B1, SW3.B2, SW4.B1, SW4.B2, U4.1, U4.10, U4.12, U4.29, U4.30, U4.8; no longer C11.2, C16.1, C18.1, C2.2, C20.2, C21.1, C22.1, C23.2, C24.1, C5.1, C7.2, CHRG2.2, J1.1, LDO2.2, LED3.C, LED4.C, R11.1, R14.1, R15.1, R7.2, SW1.B1, SW1.B2, SW2.B1, SW2.B2, SW3.1, SW4.3, U3.1, U3.10, U3.12, U3.29, U3.30, U3.8, U4.4
- net LED1: now also R4.2; no longer R3.2
- net LED2: now also R5.2; no longer R4.2
- net MOSI: now also U4.19; no longer U3.19
- net N$1: now also R13.2, U4.11; no longer R6.2, U3.11
- net N$10: now also LED2.A, R5.1; no longer LED4.A, R4.1
- net N$12: now also C1.1; no longer C7.1
- net N$13: now also C15.2, U4.28; no longer C16.2, U3.28
- net N$15: now also C17.2, U4.27; no longer C18.2, U3.27
- net N$17: now also CHRG.5, R6.2; no longer CHRG2.5, R11.2
- net N$19: now also RTC.2, XTAL2.P$1; no longer U4.2, XTAL3.P$1
- net N$2: now also R15.1, U4.26; no longer R7.1, U3.26
- net N$20: now also RTC.1, XTAL2.P$2; no longer U4.1, XTAL3.P$2
- net N$23: now also R11.2; no longer R17.2
- net N$24: now also R12.2; no longer R18.2
- net N$25: now also LED3.C, R14.2; no longer LED5.C, R19.2
- net N$26: now also LED4.C; no longer LED6.C
- net N$3: now also C18.2, U4.2; no longer C13.2, U3.2
- net N$4: now also C3.2, XTAL1.P$1; no longer C8.2, XTAL2.P$1
- net N$5: now also C18.1, U4.3; no longer C13.1, U3.3
- net N$6: now also C4.1, XTAL1.P$2; no longer C9.1, XTAL2.P$2
- net N$7: now also C16.2, U4.4; no longer C15.2, U3.4
- net N$8: now also C16.1, U4.5; no longer C15.1, U3.5
- net N$9: now also LED1.A, R4.1; no longer LED3.A, R3.1
- net P0.09/NFC1: now also C5.1; no longer C11.1
- net P0.10/NFC2: now also C6.1; no longer C10.1
- net RESET: now also C11.2, D3.+, R10.1, SW2.1; no longer C14.2, D1.+, R5.1, SW4.1
- net RXD.FT: now also R18.1; no longer R2.1
- net RXD.NRF: now also R17.2; no longer R1.2
- net RXLED: now also R14.1; no longer R19.1
- net SCK: now also U4.18; no longer U3.18
- net SCL: now also R2.1, RTC.6; no longer J1.3, R9.1, U4.6
- net SDA: now also R1.1, RTC.5; no longer J1.4, R8.1, U4.5
- net TXD.FT: now also R17.1; no longer R1.1
- net TXD.NRF: now also R18.2; no longer R2.2
- net USB+: now also C13.1, R12.1; no longer C23.1, R18.1
- net USB-: now also C12.2, R11.1; no longer C24.2, R17.1
- net VBAT: now also RTC.3; no longer U4.3
- net VIN: now also C7.2, C8.2, CHRG.4, D1.-, LDO1.1, LDO1.3, R3.2; no longer C21.2, C5.2, CHRG2.4, D4.-, LDO2.1, LDO2.3, R12.2
- net VLIPO: now also C10.1, CHRG.3, D1.+, R8.2; no longer C20.1, CHRG2.3, D4.+, R13.2

Commit message: updated through Take 005
Parts:
- removed C5, C6: 300p, LinnesLab-Passives:C0603
- moved R18 88.4 mm to (-7.44, 82.9)
- moved R17 85.3 mm to (-2.11, 82.3)
- moved FTDI 56.2 mm to (-5.61, 76.8)
- moved C14 51.0 mm to (-10.5, 78.4), turned to 270 degrees
- moved R16 50.3 mm to (-0.10, 79.9)
- moved R14 47.4 mm to (-0.13, 77.7)
- moved LED4 43.3 mm to (3.63, 79.9), turned to 180 degrees
- moved LED3 41.0 mm to (3.63, 77.7), turned to 180 degrees
- moved C12 40.2 mm to (3.71, 74.5), turned to 180 degrees
- moved R7 37.4 mm to (14.0, 1.60), flipped to the bottom, turned to 180 degrees
- moved C13 37.2 mm to (3.71, 72.6)
- moved LDO1 33.1 mm to (12.9, 4.14), flipped to the bottom, turned to 90 degrees
- moved C9 31.7 mm to (15.7, 4.06), flipped to the bottom, turned to 90 degrees
- moved C8 30.5 mm to (9.98, 4.06), flipped to the bottom, turned to 270 degrees
- moved R15 30.0 mm to (30.8, 17.7), turned to 0 degrees
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Connections:
- net GND: no longer C5.2, C6.2
- net P0.09/NFC1: no longer C5.1
- net P0.10/NFC2: no longer C6.1
Routing:
- net GND: track 0.00 -> 20.2 mm, vias 0 -> 12
- net VLIPO: track 0.00 -> 14.1 mm
- net TXLED: track 0.00 -> 12.7 mm, vias 0 -> 2
- net VIN: track 0.00 -> 7.71 mm
- net RXD.FT: track 0.00 -> 6.74 mm
- net N$2: track 0.00 -> 6.47 mm
- net N$12: track 0.00 -> 5.57 mm
- net N$13: track 0.00 -> 5.18 mm
- net N$8: track 0.00 -> 4.57 mm
- net N$5: track 0.00 -> 4.53 mm
- net 3.3V: track 0.00 -> 4.49 mm, vias 0 -> 1
- net N$15: track 0.00 -> 3.54 mm
- net N$3: track 0.00 -> 3.17 mm
- net N$7: track 0.00 -> 3.01 mm
- net TXD.FT: track 0.00 -> 2.72 mm
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- added copper zone on layer 1, net 3.3V
- added copper zone on layer 16, net GND

Commit message: updated through Take 005
Parts:
- moved R18 71.7 mm to (4.19, 12.1)
- moved FTDI 71.4 mm to (6.05, 6.38)
- moved R17 71.1 mm to (9.47, 12.2)
- moved R11 70.6 mm to (11.6, 4.85)
- moved R12 70.3 mm to (11.7, 3.23)
- moved C14 70.3 mm to (1.85, 9.19)
- moved LED4 70.2 mm to (15.3, 10.7)
- moved R16 70.1 mm to (11.6, 10.7)
- moved LED3 70.0 mm to (15.3, 8.74)
- moved R14 69.9 mm to (11.6, 8.81)
- moved C13 69.3 mm to (14.0, 4.06), turned to 90 degrees
- moved C12 67.9 mm to (14.2, 7.34)
- moved JP1 58.8 mm to (1.73, 1.96), turned to 90 degrees
- moved R2 49.8 mm to (9.73, 34.8)
- moved R1 49.3 mm to (9.78, 37.0)
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Routing:
- net USB-: track 2.15 -> 23.6 mm, vias 0 -> 1
- net TXLED: track 12.7 -> 0.00 mm, vias 2 -> 0
- net USB+: track 2.15 -> 14.4 mm, vias 0 -> 1
- net GND: track 20.2 -> 28.9 mm, vias 12 -> 14
- net VLIPO: track 14.1 -> 22.5 mm
- net N$17: track 0.00 -> 7.70 mm
- net N$4: track 0.00 -> 7.22 mm
- net N$6: track 0.00 -> 6.68 mm
- net N$2: track 6.47 -> 0.00 mm
- net VIN: track 7.71 -> 14.1 mm
- net N$13: track 5.18 -> 0.00 mm
- net N$15: track 3.54 -> 0.00 mm
- net SWDIO: track 0.00 -> 1.48 mm, vias 0 -> 1
- net RXLED: track 1.96 -> 2.62 mm
