File: Hardware/Basic/Bottom/NotSoSmartWatch-BASIC-BOTTOM-version2.sch (EAGLE design)
At the start: 45 parts, among them U1 AD5242-SO16

Commit message: updated through Take 007
Parts:
- removed C4, C7: 4.7u, LinnesLab-Passives:CAPACITOR0603
- removed C8, C9: 1u, LinnesLab-Passives:CAPACITOR0603
- removed CHRG: MCP73831, LinnesLab-Power:MCP73831
- removed LDO1: MIC5504, LinnesLab-Power:MIC5504
- removed R3, R7: 100k, LinnesLab-Passives:RESISTOR0603
- removed R6: (no value), LinnesLab-Passives:RESISTOR0603
Connections:
- removed net D27/CHRG.STAT: CHRG.STAT, R3.1
- removed net N$14: CHRG.PROG, R6.2
- removed net VIN1: C7.2, C8.2, CHRG.VIN, LDO1.EN, LDO1.IN, R3.2
- removed net VLIPO: C4.1, CHRG.VBAT
- new net A4/PPG: J1.7
- new net A5/TIA: J1.6
- new net D30/LED.CTRL: J1.5
- net 3.3V: now also J1.4; no longer C9.1, J1.7, LDO1.OUT, R7.2
- net A6/TIA: no longer J1.3
- net A7/PPG: no longer J1.4
- net D29/LED.CTRL: no longer J1.5
- net GND: now also J1.3; no longer C4.2, C7.1, C8.1, C9.2, CHRG.VSS, J1.6, LDO1.GND, R6.1, R7.1

Commit message: updated through Take 008
Connections:
- removed net A6/TIA: C10.2, C15.1, OP4G$1.OUT, U1.W1
- removed net A7/PPG: C21.2, OP3G$1.OUT, U1.B2
- removed net D29/LED.CTRL: U$4.A
- net A4/PPG: now also C21.2, OP3G$1.OUT, U1.B2
- net A5/TIA: now also C10.2, C15.1, OP4G$1.OUT, U1.W1
- net D30/LED.CTRL: now also U$4.A
Changed lines of the file:
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@@
-</segment>
-</net>
-<net name="A6/TIA" class="0">
-<segment>
-<wire x1="154.94" y1="43.18" x2="149.86" y2="43.18" width="0.1524" layer="91"/>
-<label x="149.86" y="43.18" size="1.27" layer="95" rot="R180" xref="yes"/>
-<pinref part="U1" gate="G$1" pin="W1"/>
-</segment>
-<segment>
-<pinref part="C10" gate="G$1" pin="2"/>
-<wire x1="81.28" y1="134.62" x2="88.9" y2="134.62" width="0.1524" layer="91"/>
-<wire x1="88.9" y1="134.62" x2="88.9" y2="124.46" width="0.1524" layer="91"/>
-<wire x1="88.9" y1="134.62" x2="88.9" y2="144.78" width="0.1524" layer="91"/>
-<junction x="88.9" y="134.62"/>
-<label x="88.9" y="144.78" size="1.27" layer="95" rot="R180" xref="yes"/>
-<pinref part="C15" gate="G$1" pin="1"/>
-<wire x1="91.44" y1="124.46" x2="88.9" y2="124.46" width="0.1524" layer="91"/>
-<pinref part="OP4" gate="G$1" pin="OUT"/>
-<wire x1="86.36" y1="124.46" x2="88.9" y2="124.46" width="0.1524" layer="91"/>
-<junction x="88.9" y="124.46"/>
 </segment>
 </net>
@@
 </segment>
 </net>
-<net name="D29/LED.CTRL" class="0">
-<segment>
-<pinref part="U$4" gate="G$1" pin="A"/>
-<wire x1="248.92" y1="45.72" x2="251.46" y2="45.72" width="0.1524" layer="91"/>
-<wire x1="251.46" y1="45.72" x2="251.46" y2="53.34" width="0.1524" layer="91"/>
-<label x="251.46" y="53.34" size="1.27" layer="95" rot="R180" xref="yes"/>
-</segment>
-</net>
 <net name="N$10" class="0">
 <segment>
@@
 <wire x1="71.12" y1="40.64" x2="71.12" y2="38.1" width="0.1524" layer="91"/>
 <junction x="71.12" y="40.64"/>
-</segment>
-</net>
-<net name="A7/PPG" class="0">
-<segment>
-<wire x1="182.88" y1="43.18" x2="185.42" y2="43.18" width="0.1524" layer="91"/>
-<label x="185.42" y="43.18" size="1.27" layer="95" xref="yes"/>
-<pinref part="U1" gate="G$1" pin="B2"/>
-</segment>
-<segment>
-<pinref part="C21" gate="G$1" pin="2"/>
-<wire x1="220.98" y1="127" x2="228.6" y2="127" width="0.1524" layer="91"/>
-<wire x1="228.6" y1="127" x2="228.6" y2="116.84" width="0.1524" layer="91"/>
-<pinref part="OP3" gate="G$1" pin="OUT"/>
-<wire x1="228.6" y1="116.84" x2="226.06" y2="116.84" width="0.1524" layer="91"/>
-<wire x1="228.6" y1="127" x2="228.6" y2="137.16" width="0.1524" layer="91"/>
-<junction x="228.6" y="127"/>
-<label x="228.6" y="137.16" size="1.27" layer="95" rot="R180" xref="yes"/>
-<label x="228.6" y="116.84" size="1.27" layer="95" xref="yes"/>
 </segment>
 </net>
@@
 <label x="162.56" y="-20.32" size="1.016" layer="95" xref="yes"/>
 </segment>
+<segment>
+<pinref part="U$4" gate="G$1" pin="A"/>
+<wire x1="248.92" y1="45.72" x2="251.46" y2="45.72" width="0.1524" layer="91"/>
+<wire x1="251.46" y1="45.72" x2="251.46" y2="53.34" width="0.1524" layer="91"/>
+<label x="251.46" y="53.34" size="1.27" layer="95" rot="R180" xref="yes"/>
+</segment>
 </net>
 <net name="A5/TIA" class="0">
@@
 <label x="162.56" y="-17.78" size="1.016" layer="95" xref="yes"/>
 </segment>
+<segment>
+<pinref part="C10" gate="G$1" pin="2"/>
+<wire x1="81.28" y1="134.62" x2="88.9" y2="134.62" width="0.1524" layer="91"/>
+<wire x1="88.9" y1="134.62" x2="88.9" y2="124.46" width="0.1524" layer="91"/>
+<wire x1="88.9" y1="134.62" x2="88.9" y2="144.78" width="0.1524" layer="91"/>
+<junction x="88.9" y="134.62"/>
+<label x="88.9" y="144.78" size="1.27" layer="95" rot="R180" xref="yes"/>
+<pinref part="C15" gate="G$1" pin="1"/>
+<wire x1="91.44" y1="124.46" x2="88.9" y2="124.46" width="0.1524" layer="91"/>
+<pinref part="OP4" gate="G$1" pin="OUT"/>
+<wire x1="86.36" y1="124.46" x2="88.9" y2="124.46" width="0.1524" layer="91"/>
+<junction x="88.9" y="124.46"/>
+</segment>
+<segment>
+<wire x1="154.94" y1="43.18" x2="149.86" y2="43.18" width="0.1524" layer="91"/>
+<label x="149.86" y="43.18" size="1.27" layer="95" rot="R180" xref="yes"/>
+<pinref part="U1" gate="G$1" pin="W1"/>
+</segment>
 </net>
 <net name="A4/PPG" class="0">
@@
 <label x="162.56" y="-15.24" size="1.016" layer="95" xref="yes"/>
 </segment>
-</net>
+<segment>
+<pinref part="C21" gate="G$1" pin="2"/>
+<wire x1="220.98" y1="127" x2="228.6" y2="127" width="0.1524" layer="91"/>
+<wire x1="228.6" y1="127" x2="228.6" y2="116.84" width="0.1524" layer="91"/>
+<pinref part="OP3" gate="G$1" pin="OUT"/>
+<wire x1="228.6" y1="116.84" x2="226.06" y2="116.84" width="0.1524" layer="91"/>
+<wire x1="228.6" y1="127" x2="228.6" y2="137.16" width="0.1524" layer="91"/>
+<junction x="228.6" y="127"/>
+<label x="228.6" y="137.16" size="1.27" layer="95" rot="R180" xref="yes"/>
+<label x="228.6" y="116.84" size="1.27" layer="95" xref="yes"/>
+</segment>
+<segment>
+<wire x1="182.88" y1="43.18" x2="185.42" y2="43.18" width="0.1524" layer="91"/>
+<label x="185.42" y="43.18" size="1.27" layer="95" xref="yes"/>
+<pinref part="U1" gate="G$1" pin="B2"/>
+</segment>
+</net>
