File: Hardware/Basic/Bottom/NotSoSmartWatch-BASIC-BOTTOM-version2.brd (EAGLE design)
At the start: 33 x 33 mm, 45 parts, among them U1 AD5242-SO16

Commit message: updated through Take 007
Parts:
- removed C4, C7: 4.7u, LinnesLab-Passives:C0603
- removed C8, C9: 1u, LinnesLab-Passives:C0603
- removed CHRG: MCP73831, LinnesLab-Power:SOT23-5
- removed LDO1: MIC5504, LinnesLab-Power:SOT23-5
- removed R3, R7: 100k, LinnesLab-Passives:R0603
- removed R6: (no value), LinnesLab-Passives:R0603
- moved J1 1.27 mm to (5.08, 33.0)
Connections:
- removed net D27/CHRG.STAT: CHRG.1, R3.1
- removed net N$14: CHRG.5, R6.2
- removed net VIN1: C7.2, C8.2, CHRG.4, LDO1.1, LDO1.3, R3.2
- removed net VLIPO: C4.1, CHRG.3
- new net A4/PPG: J1.7
- new net A5/TIA: J1.6
- new net D30/LED.CTRL: J1.5
- net 3.3V: now also J1.4; no longer C9.1, J1.7, LDO1.5, R7.2
- net A6/TIA: no longer J1.3
- net A7/PPG: no longer J1.4
- net D29/LED.CTRL: no longer J1.5
- net GND: now also J1.3; no longer C4.2, C7.1, C8.1, C9.2, CHRG.2, J1.6, LDO1.2, R6.1, R7.1
Routing:
- net SDA: track 49.6 -> 4.82 mm, vias 2 -> 0
- net A6/TIA: track 64.8 -> 39.3 mm
- net SCL: track 48.0 -> 27.9 mm
- net A7/PPG: track 39.4 -> 19.9 mm
- net D29/LED.CTRL: track 9.24 -> 0.00 mm
- net N$9: track 4.17 -> 3.12 mm

Commit message: updated through Take 008 - one airwire I don't understand, hopefully no polygon issues but not sure, drill clearance??:
Parts:
- moved C3 57.2 mm to (33.6, 31.1), turned to 270 degrees
- moved XTAL2 55.5 mm to (24.7, 31.8), turned to 90 degrees
- moved RTC 52.7 mm to (29.0, 30.6)
- moved C17 22.6 mm to (5.90, 17.0)
- moved U$4 17.4 mm to (6.69, 19.6), turned to 180 degrees
- moved C2 4.09 mm to (30.8, 24.6), turned to 180 degrees
- moved C1 1.51 mm to (6.96, 22.8)
- moved IMU1 1.51 mm to (7.14, 27.2)
- moved C18 0.60 mm to (5.90, 9.04)
Connections:
- removed net A6/TIA: C10.2, C15.1, OP4.1, U1.3
- removed net A7/PPG: C21.2, OP3.1, U1.14
- removed net D29/LED.CTRL: U$4.8
- net A4/PPG: now also C21.2, OP3.1, U1.14
- net A5/TIA: now also C10.2, C15.1, OP4.1, U1.3
- net D30/LED.CTRL: now also U$4.8
Routing:
- net SDA: track 4.82 -> 82.0 mm, vias 0 -> 1
- net A5/TIA: track 0.00 -> 63.0 mm, vias 0 -> 3
- net A4/PPG: track 0.00 -> 40.0 mm, vias 0 -> 1
- net A6/TIA: track 39.3 -> 0.00 mm, vias 2 -> 0
- net SCL: track 27.9 -> 63.2 mm, vias 0 -> 2
- net N$9: track 3.12 -> 25.9 mm, vias 0 -> 2
- net A7/PPG: track 19.9 -> 0.00 mm
- net D30/LED.CTRL: track 0.00 -> 15.6 mm
- net GND: track 29.2 -> 34.5 mm, vias 13 -> 16
- net N$11: track 0.00 -> 1.77 mm
- net N$12: track 0.00 -> 1.69 mm
- net VREF: track 37.4 -> 36.9 mm
